File: venta_overdrive.kicad_sch (KiCad schematic)
At the start: 48 parts, among them J1 IN, J2 OUT, J3 9V, J4 GND, J5 GND, J6 LED-, U1 JRC4558D, U2 JRC4558D, U3 JRC4558D

Commit message: use external LED
Parts:
- removed C12: 100n, Capacitor_SMD:C_0805_2012Metric, symbol Venta:C
- removed C2: 10u, Capacitor_SMD:C_0805_2012Metric, symbol Venta:C
- removed C4, C9: 220n, Capacitor_SMD:C_0805_2012Metric, symbol Venta:C
- removed C5: 680n, Capacitor_SMD:C_0805_2012Metric, symbol Venta:C
- removed R15: 100k, Resistor_SMD:R_0805_2012Metric, symbol Venta:R
- removed R16: 1k, Resistor_SMD:R_0805_2012Metric, symbol Venta:R
- removed R17: 3.3k, Resistor_SMD:R_0805_2012Metric, symbol Venta:R
- removed R3: 1M, Resistor_SMD:R_0805_2012Metric, symbol Venta:R
- removed RV1: B50k Drive, Venta:Pot_Alpha_16mm_RA_Single, symbol Venta:POT
- removed RV2: B50k Resonance, Venta:Pot_Alpha_16mm_RA_Single, symbol Venta:POT
- removed unit 1 of RV3
- removed unit 2 of U2
- removed unit 1 of U3
- added C1: 22u, Capacitor_SMD:C_1206_3216Metric, symbol Venta:C
- added C7: 1.5n, Capacitor_SMD:C_0603_1608Metric, symbol Venta:C
- added D3: SS14, Diode_SMD:D_SMA, symbol Venta:D_Schottky
- added J7: GND, Venta:WirePad, symbol Venta:PAD
- added R10, R9: 33k, Resistor_SMD:R_0805_2012Metric, symbol Venta:R
- added R12, R13: 15k, Resistor_SMD:R_0805_2012Metric, symbol Venta:R
- added R4: 220k, Resistor_SMD:R_0805_2012Metric, symbol Venta:R
- added unit 2 of RV3
- added unit 1 of U1
- added unit 3 of U1
- added V2: VDC, symbol Venta:VSOURCE
- C10: renamed from U2; value JRC4558D -> 100n; footprint Package_SO:SOIC-8_3.9x4.9mm_P1.27mm -> Capacitor_SMD:C_0805_2012Metric; symbol Venta:OPAMP_DUAL -> Venta:C; LCSC C443686 -> C49678; Note U2A summer, U2B integrator 1 -> U1 decoupling (new)
- C11: renamed from U3; value JRC4558D -> 100n; footprint Package_SO:SOIC-8_3.9x4.9mm_P1.27mm -> Capacitor_SMD:C_0805_2012Metric; symbol Venta:OPAMP_DUAL -> Venta:C; LCSC C443686 -> C49678; Note U3A Vref buffer, U3B integrator 2 -> U2 decoupling (new)
- C12: renamed from C10; Note U1 decoupling (new) -> U3 decoupling (new)
- C2: renamed from R1; value 10k -> 10u; footprint Resistor_SMD:R_0805_2012Metric -> Capacitor_SMD:C_0805_2012Metric; symbol Venta:R -> Venta:C; LCSC C17414 -> C15850; Note (none) -> 25V X5R
- C3: renamed from J6; value LED- -> 22n; footprint Venta:WirePad -> Capacitor_SMD:C_0805_2012Metric; symbol Venta:PAD -> Venta:C; LCSC (none) -> C1729; Note to 3PDT LED lug -> (none)
- C4: renamed from C3; value 22n -> 220n; LCSC C1729 -> C5378
- C5: renamed from U1; value JRC4558D -> 680n; footprint Package_SO:SOIC-8_3.9x4.9mm_P1.27mm -> Capacitor_SMD:C_0805_2012Metric; symbol Venta:OPAMP_DUAL -> Venta:C; LCSC C443686 -> C107133; Note U1A gain, U1B input buffer -> 50V X7R
- C8: renamed from R13; value 15k -> 220n; footprint Resistor_SMD:R_0805_2012Metric -> Capacitor_SMD:C_0805_2012Metric; symbol Venta:R -> Venta:C; LCSC C17475 -> C5378
- J6: renamed from C11; value 100n -> LED+; footprint Capacitor_SMD:C_0805_2012Metric -> Venta:WirePad; symbol Venta:C -> Venta:PAD; LCSC C49678 -> (none); Note U2 decoupling (new) -> to the external LED anode (LED has its own resistor)
- R1: renamed from D3; value SS14 -> 10k; footprint Diode_SMD:D_SMA -> Resistor_SMD:R_0805_2012Metric; symbol Venta:D_Schottky -> Venta:R; LCSC C2480 -> C17414; Note reverse-polarity protection (was 1N5817) -> (none)
- R11: renamed from R9; value 33k -> 3k; LCSC C17633 -> C17661
- R14: renamed from C7; value 1.5n -> 3.3k; footprint Capacitor_SMD:C_0603_1608Metric -> Resistor_SMD:R_0805_2012Metric; symbol Venta:C -> Venta:R; LCSC C107039 -> C26010; Note C0G/NP0 -> (none)
- R15: renamed from R14; value 3.3k -> 100k; LCSC C26010 -> C149504
- R16: renamed from RV4; value B50k Volume -> 1k; footprint Venta:Pot_Alpha_16mm_RA_Single -> Resistor_SMD:R_0805_2012Metric; symbol Venta:POT -> Venta:R; LCSC (none) -> C17513
- R2: renamed from C1; value 22u -> 10k; footprint Capacitor_SMD:C_1206_3216Metric -> Resistor_SMD:R_0805_2012Metric; symbol Venta:C -> Venta:R; LCSC C12891 -> C17414; Note bulk, 25V X5R (was 47u electrolytic) -> (none)
- R3: renamed from D4; value LED red 5mm -> 1M; footprint LED_THT:LED_D5.0mm -> Resistor_SMD:R_0805_2012Metric; symbol Venta:LED -> Venta:R; LCSC (none) -> C17514; Note hand-solder; cathode goes to 3PDT -> input pulldown (was 1.5M)
- RV1: renamed from R4; value 220k -> B50k Drive; footprint Resistor_SMD:R_0805_2012Metric -> Venta:Pot_Alpha_16mm_RA_Single; symbol Venta:R -> Venta:POT; LCSC C17556 -> (none)
- RV2: renamed from R10; value 33k -> B50k Resonance; footprint Resistor_SMD:R_0805_2012Metric -> Venta:Pot_Alpha_16mm_RA_Single; symbol Venta:R -> Venta:POT; LCSC C17633 -> (none)
- RV3: renamed from R11; value 3k -> B50k dual Eq; footprint Resistor_SMD:R_0805_2012Metric -> Venta:Pot_Alpha_16mm_RA_Dual; symbol Venta:R -> Venta:POT_DUAL; LCSC C17661 -> (none)
- RV4: renamed from U3; value JRC4558D -> B50k Volume; footprint Package_SO:SOIC-8_3.9x4.9mm_P1.27mm -> Venta:Pot_Alpha_16mm_RA_Single; symbol Venta:OPAMP_DUAL -> Venta:POT; LCSC C443686 -> (none); Note U3A Vref buffer, U3B integrator 2 -> (none)
- U2: renamed from V2; value VDC -> JRC4558D; footprint (none) -> Package_SO:SOIC-8_3.9x4.9mm_P1.27mm; symbol Venta:VSOURCE -> Venta:OPAMP_DUAL; LCSC (none) -> C443686; Note (none) -> U2A summer, U2B integrator 1; now in the parts list
- U2: renamed from R12; value 15k -> JRC4558D; footprint Resistor_SMD:R_0805_2012Metric -> Package_SO:SOIC-8_3.9x4.9mm_P1.27mm; symbol Venta:R -> Venta:OPAMP_DUAL; LCSC C17475 -> C443686; Note (none) -> U2A summer, U2B integrator 1
- U3: renamed from U1; Note U1A gain, U1B input buffer -> U3A Vref buffer, U3B integrator 2
- U3: renamed from RV3; value B50k dual Eq -> JRC4558D; footprint Venta:Pot_Alpha_16mm_RA_Dual -> Package_SO:SOIC-8_3.9x4.9mm_P1.27mm; symbol Venta:POT_DUAL -> Venta:OPAMP_DUAL; LCSC (none) -> C443686; Note (none) -> U3A Vref buffer, U3B integrator 2
- U3: renamed from R2; value 10k -> JRC4558D; footprint Resistor_SMD:R_0805_2012Metric -> Package_SO:SOIC-8_3.9x4.9mm_P1.27mm; symbol Venta:R -> Venta:OPAMP_DUAL; LCSC C17414 -> C443686; Note (none) -> U3A Vref buffer, U3B integrator 2
- renumbered C8 to C9
Connections:
- net LED_A is gone; now on net GND: R3.2
- net LED_K is gone; now on net IN: C3.1, R3.1
- net +9V_IN: now also D3.2 (A), V2.1 (+); no longer R1.2 (A), U2.1 (+)
- net BP: now also RV2.3, U2.7, RV3.6; no longer U3.6
- net BUF_IN: now also C3.2, R4.1; no longer C4.2, RV1.1
- net BUF_OUT: now also C4.1
- net DRIVE_HI: now also C4.2, RV1.3
- net DRIVE_W: now also RV1.2, U1.3 (+); no longer C5.3 (+)
- net EQ_A: now also RV3.3, R12.2; no longer U2.2
- net EQ_B: now also R13.1, RV3.4, RV3.5; no longer C8.1, U3.4, U3.5
- net GAIN_FB: now also U1.2 (-); no longer C5.2 (-)
- net GAIN_OUT: now also U1.1; no longer C5.1
- net GAIN_RC: now also C5.1
- net GND: now also C10.2, C11.2, C2.2, R15.2, RV4.1, U2.4 (V-), C1.2, J7.1, U1.4 (V-), V2.2 (-); no longer C10.4 (V-), C11.4 (V-), J6.2, R16.1, U2.2 (-), U3.2
- net HP: now also R12.1, R9.2; no longer R11.2, U2.1
- net IN: no longer C4.1
- net INT1_N: now also RV3.1, RV3.2, U2.6 (-)
- net INT2_N: now also U3.6 (-), C7.2, R13.2; no longer C8.2, R14.2, RV4.6 (-)
- net LP: now also C8.1, U3.7, C7.1, R10.2; no longer C9.1, R14.1, RV2.2, RV4.7
- net LP_AC: now also C8.2, R14.1; no longer C9.2, R15.1
- net OUT: now also R16.2
- net OUT_DC: now also C9.2, R15.1, R16.1
- net RES: now also R11.1, RV2.1, RV2.2; no longer RV3.1
- net SUM: now also R10.1, R9.1; no longer R11.1, RV2.1
- net VB: now also C2.1, R1.2, R2.1, U3.3 (+); no longer C2.2, U3.1
- net VCC: now also C10.1, C11.1, U2.8 (V+), C1.1, D3.1 (K), U1.8 (V+); no longer C10.8 (V+), C11.8 (V+), C2.1, R2.1
- net VOL_HI: now also R14.2, RV4.3; no longer R15.2, R16.3
- net VOL_W: now also C9.1, RV4.2; no longer R16.2
- net VREF: now also C5.2, R11.2, RV1.1, U2.5 (+), U3.1, U3.2 (-), U3.5 (+), R4.2; no longer RV1.2, RV3.2, RV4.5 (+)
Other:
- note added: "Power, reference voltage VREF = VCC/2, external LED pads"
- note added: "V1 (100 mV, 440 Hz sine) and V2 (9 V) are for simulation only and are not on the board. J1..J7: wire pads for the jacks, the footswitch and the external LED."
- note removed: "Power, reference voltage VREF = VCC/2, LED"
- note removed: "V1 (100 mV, 440 Hz sine) and V2 (9 V) are for simulation only and are not on the board. J1..J6: wire pads for the jacks and the footswitch."
- moved on the sheet: C10, C11, C12, C4, C9, R11, R15, RV4, U3B, U3C
