File: venta_overdrive.kicad_sch (KiCad schematic)
At the start: 47 parts, among them J1 IN, J2 OUT, J3 9V, J4 GND, J5 GND, J6 LED+, J7 GND, U1 JRC4558D, U2 JRC4558D, U3 JRC4558D

Commit message: fix R8 nominal
Parts:
- R8: value 15k -> 75k; LCSC C17475 -> C17819; Note (none) -> 75k as in the factory schematic (the stripboard layout has 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
Changed lines of the file:
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@@
 			)
 		)
-		(property "Value" "15k"
+		(property "Value" "75k"
 			(at 55.88 237.49 0)
 			(show_name no)
@@
 			)
 		)
-		(property "LCSC" "C17475"
+		(property "LCSC" "C17819"
 			(at 53.34 236.22 0)
 			(hide yes)
+			(show_name no)
+			(do_not_autoplace no)
+			(effects
+				(font
+					(size 1.27 1.27)
+				)
+			)
+		)
+		(property "Note" "75k as in the factory schematic (the stripboard layout has 15k)"
+			(at 53.34 236.22 0)
+			(hide yes)

Commit message: fix Resonance direction
Connections:
- net BP: now also RV2.1; no longer RV2.3
- net RES: now also RV2.3; no longer RV2.1
Changed lines of the file:
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@@
 		)
 	)
-	(label "RES"
+	(label "BP"
 		(at 212.09 229.87 90)
 		(effects
@@
 		)
 	)
-	(label "BP"
+	(label "RES"
 		(at 212.09 242.57 270)
 		(effects
